File: hardware/MRC/mrc_adc.kicad_sch (KiCad schematic)
At the start: 37 parts, among them U16 TPS79618, U4 LT6600-xx, U5 LTC2145-14, U8 LT6600-xx

Commit message: well scanning, AFE
Parts:
- renumbered C8 to C10, C8 to C133, C22 to C157, C22 to C158, C22 to C159, C22 to C160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
