File: hardware/MRC/mrc_adc.kicad_sch (KiCad schematic)
At the start: 37 parts, among them U16 TPS79618, U4 LT6600-xx, U5 LTC2145-14, U8 LT6600-xx

Commit message: Update KiCAD Version, Integrate Libraries
Parts:
- renumbered C8 to C10, C8 to C133, C22 to C157, C22 to C158, C22 to C159, C22 to C160, C22 to C161, C22 to C162, C1 to C2, C2 to C3, C8 to C37, C8 to C39, C8 to C6, C6 to C7, C8 to C89, C7 to C9, C8 to C90, C8 to C91, C8 to C92, C8 to C93, C8 to C94, C8 to C95, R44 to R17, R44 to R18, R44 to R19, R44 to R20, R44 to R21, R44 to R22, R44 to R23, R44 to R7

Commit message: Clean bill of materials
Parts:
- C10, C133, C162, C93, C94, C95: MPN (none) -> C0603C104K1RACAUTO
- C157, C161: MPN (none) -> KGM15CR51A106MT
- C158, C2, C3, C7, C89, C9, C91: MPN (none) -> KAM15AR72A103KT
- C159: MPN (none) -> KGM15BR51A475KT
- C37, C39: MPN (none) -> KGM15ACG1H180JT
- C6: MPN (none) -> KGM15BR50J225KT
- C90, C92: MPN (none) -> KGM15BR51E105KM
- FB15: MPN (none) -> 742792641
- R17, R18, R19, R7: MPN (none) -> KTR03EZPF49R9
- R31: MPN (none) -> CMP0603AFX-1002L
- U16: MPN (none) -> TPS79618DCQR
- U4, U8: MPN (none) -> LT6600IS8-20#PBF
- U5: MPN (none) -> LTC2145CUP-14#PBF
