File: hardware/MRC/mrc_adc.kicad_sch (KiCad schematic)
At the start: 37 parts, among them U16 TPS79618, U4 LT6600-xx, U5 LTC2145-14, U8 LT6600-xx

Commit message: KiCAD schematic modification
Parts:
- added C168, C169, C189, C193, C194: 100n, Capacitor_SMD:C_0603_1608Metric, symbol Device:C_Small
- added U25: USBLC6-4SC6, Package_TO_SOT_SMD:SOT-23-6, symbol Power_Protection:USBLC6-4SC6
- C10, C133, C162, C93, C94, C95: MPN C0603C104K1RACAUTO -> C14663
- C157, C161: MPN KGM15CR51A106MT -> C96446
- C158, C2, C3, C7, C89, C9, C91: MPN KAM15AR72A103KT -> C57112
- C159: MPN KGM15BR51A475KT -> C19666
- C160: MPN (none) -> C4978585; Stock (none) -> Extended
- C37, C39: MPN KGM15ACG1H180JT -> C1647
- C6: MPN KGM15BR50J225KT -> C23630
- C8: MPN W2L14Z225MAT1S -> C23630
- C90, C92: MPN KGM15BR51E105KM -> C15849
- FB15: MPN 742792641 -> C14709
- R17, R18, R19, R7: MPN KTR03EZPF49R9 -> C23185
- R20, R21, R22, R23: MPN (none) -> C23049; Stock (none) -> Extended
- R31: MPN CMP0603AFX-1002L -> C25804
- U16: MPN TPS79618DCQR -> C2867020; Stock (none) -> Extended
- U4, U8: MPN LT6600IS8-20#PBF -> C673220/C107980/C673198/C673202/C673216; Stock (none) -> Extended
- U5: MPN LTC2145CUP-14#PBF -> C679368/C679372; Stock (none) -> Extended
Connections:
- net +3V3: now also C194.2, U25.5 (VBUS)
- net ADC_AINA: now also C169.1, U25.1 (I/O1); no longer R23.2
- net ADC_AINB: now also C193.1, U25.3 (I/O2); no longer R21.2
- net GND: now also C168.1, C189.1, C194.1, U25.2 (GND); no longer R20.1, R22.1
- new net: C168.2, R22.1
- new net: C193.2, R21.2
- new net: C169.2, R23.2
- new net: C189.2, R20.1
Other:
- moved on the sheet: C93
