File: hardware/MRC/mrc_clocks.kicad_sch (KiCad schematic)
At the start: 8 parts, among them U3 XLH736120.000000I, U7 LMK1D1204P

Commit message: well scanning, AFE
Parts:
- U3: value XLH736120.000000I -> XLH736120.000000I
- renumbered C22 to C108, C22 to C190, C22 to C191, C22 to C192, FB15 to FB2
