File: hardware/MRC/mrc_clocks.kicad_sch (KiCad schematic)
At the start: 8 parts, among them U3 XLH736120.000000I, U7 LMK1D1204P

Commit message: KiCAD schematic modification
Parts:
- C108, C191: MPN KGM15BR51E105KM -> C15849
- C190: MPN KGM15CR51A106MT -> C96446
- C192: MPN C0603C104K1RACAUTO -> C14663
- FB2: MPN 742792641 -> C14709
- R6: MPN CRCW06031K00DHEBP -> C21190
- U3: MPN XLH736120.000000I -> C1670379; Stock (none) -> Extended
- U7: MPN LMK1D1204PRHDR -> C3613664; Stock (none) -> Extended
