File: hardware/MRC/mrc_dac.kicad_sch (KiCad schematic)
At the start: 75 parts, among them U1 DAC5687IPZP

Commit message: well scanning, AFE
Parts:
- renumbered C27 to C12, C33 to C14, C32 to C15, C31 to C16, C30 to C17, C88 to C24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
