File: hardware/MRC/mrc_dac.kicad_sch (KiCad schematic)
At the start: 75 parts, among them U1 DAC5687IPZP

Commit message: KiCAD schematic modification
Parts:
- C12: MPN KGM15ACG2A100FT -> C1634
- C14, C24, C27, C43, C44, C46, C47, C49, C50, C51, C52, C53, C54, C55, C56, C57, C58, C59, C60, C62, C63, C64, C86: MPN C0603C104K1RACAUTO -> C14663
- C15, C61, C73, C74, C75, C78, C82: MPN KAM15AR72A103KT -> C57112
- C16: MPN KGM15BR71E333KT -> C21117
- C17: MPN KGM15AR71E331KT -> C1664
- C28, C29, C45, C48, C65, C66, C67, C71, C72, C85: MPN KGM15CR51A106MT -> C96446
- C68, C69, C70, C76, C77: MPN KGM15BR51E105KM -> C15849
- C79, C80, C81, C83, C84: MPN KGM15CR50J476MT -> C318632; Stock (none) -> Extended
- FB5, FB6, FB7, FB8, FB9: MPN 742792641 -> C14709
- R10, R11, R14, R15: MPN SDR03EZPF51R0 -> C23197
- R12: MPN ESR03EZPJ220 -> C23345
- R16, R28: MPN SDR03EZPD1000 -> C22775
- R8: MPN CMP0603AFX-10R0L -> C22859
- R9: MPN CRCW0603-93.1-E3 -> C23132
- RBIAS1: MPN CRCW06031K00DHEBP -> C21190
- RN3, RN4, RN5, RN6: MPN EXB-2HV470JV -> C713462; Stock (none) -> Extended
- TR1, TR2: MPN ADTT1-6 -> C6495091; Stock (none) -> Extended
- U1: MPN DAC5687IPZP -> C1554572; Stock (none) -> Extended
