File: hardware/MRC/mrc_power.kicad_sch (KiCad schematic)
At the start: 37 parts, among them J12 ASMPR45-1X2-RK, J19 Conn_01x02, J20 Conn_01x02, J21 Conn_01x02, U14 LM7805_TO220, U18 LM1085-12, U19 LD29300, U20 LD29300, U21 MCP1827T-ADJ

Commit message: well scanning, AFE
Parts:
- renumbered C26 to C170, C26 to C171, R35 to R1, R35 to R100, R35 to R101, R35 to R102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
