File: hardware/MRC/mrc_power.kicad_sch (KiCad schematic)
At the start: 37 parts, among them J12 ASMPR45-1X2-RK, J19 Conn_01x02, J20 Conn_01x02, J21 Conn_01x02, U14 LM7805_TO220, U18 LM1085-12, U19 LD29300, U20 LD29300, U21 MCP1827T-ADJ

Commit message: Update KiCAD Version, Integrate Libraries
Parts:
- renumbered C26 to C170, C26 to C171, R35 to R1, R35 to R100, R35 to R101, R35 to R102, R35 to R95, R35 to R96, R35 to R97, R35 to R98, R35 to R99

Commit message: Clean bill of materials
Parts:
- C11: MPN (none) -> KGM15BR51A475KT
- C134, C154, C197, C5: MPN (none) -> KGM15BR71H334KT
- C135, C136, C199: MPN (none) -> KGM21AR50J106KU
- C137, C155: MPN (none) -> KGM15BR51E105KM
- C170, C171: MPN (none) -> KAM15BR71E224KT
- C201: MPN (none) -> KGM15CR51A106MT
- D7: MPN (none) -> ASCKC500NW5X4040
- J12: MPN (none) -> ASMPR45-1X2-RK
- R1: MPN (none) -> SDR03EZPF6201
- R100, R96: MPN (none) -> ERA-3ARB332V
- R101: MPN (none) -> CMP0603AFX-1002L
- R102: MPN (none) -> ERA-3AED203V
- R95: MPN (none) -> ERJ-UP3F5621V
- R97: MPN (none) -> CRCW06031K00DHEBP
- R98: MPN (none) -> ESR03EZPD2201
- R99: MPN (none) -> SDR03EZPD4701
- U14: MPN (none) -> LM7805CT/NOPB
- U18: MPN (none) -> LM1085IT-12/NOPB
- U19, U20: MPN (none) -> LD29300P2MTR
- U21: MPN (none) -> MCP1827T-ADJE/ET
