File: hardware/MRC/mrc_power.kicad_sch (KiCad schematic)
At the start: 37 parts, among them J12 ASMPR45-1X2-RK, J19 Conn_01x02, J20 Conn_01x02, J21 Conn_01x02, U14 LM7805_TO220, U18 LM1085-12, U19 LD29300, U20 LD29300, U21 MCP1827T-ADJ

Commit message: KiCAD schematic modification
Parts:
- C11: MPN KGM15BR51A475KT -> C19666
- C134, C154, C197, C5: MPN KGM15BR71H334KT -> C76621; Stock (none) -> Extended
- C135, C136, C199: MPN KGM21AR50J106KU -> C96446
- C137, C155: MPN KGM15BR51E105KM -> C15849
- C139, C198, C200: MPN 870575774003 -> C318632; Stock (none) -> Extended
- C170, C171: MPN KAM15BR71E224KT -> C21120
- C201: MPN KGM15CR51A106MT -> C96446
- D7: MPN ASCKC500NW5X4040 -> C2286
- J12: MPN ASMPR45-1X2-RK -> C3683033; Stock (none) -> Extended
- R1: MPN SDR03EZPF6201 -> C4260
- R100, R96: MPN ERA-3ARB332V -> C22978
- R101: MPN CMP0603AFX-1002L -> C25804
- R102: MPN ERA-3AED203V -> C4184
- R95: MPN ERJ-UP3F5621V -> C23188; Stock (none) -> Extended
- R97: MPN CRCW06031K00DHEBP -> C21190
- R98: MPN ESR03EZPD2201 -> C4190
- R99: MPN SDR03EZPD4701 -> C23162
- U14: MPN LM7805CT/NOPB -> C50931; Stock (none) -> Extended
- U18: MPN LM1085IT-12/NOPB -> C130908; Stock (none) -> Extended
- U19, U20: MPN LD29300P2MTR -> C500927; Stock (none) -> Extended
- U21: MPN MCP1827T-ADJE/ET -> C632715(no stock); Stock (none) -> Extended
