File: hardware/MRC/mrc-fpga-config.kicad_sch (KiCad schematic)
At the start: 58 parts, among them J13 Conn_02x07_Odd_Even, U15 IS25LP256D-RMLE-TR, U2 XC7A35T-FTG256

Commit message: Clean bill of materials
Parts:
- C150, C175, C176, C177, C18, C181, C182, C183, C184, C185, C19, C20, C26, C30, C31, C35, C38, C87, C88: MPN (none) -> 06035C474KAT4A
- C172, C173, C178, C179, C186, C187, C21, C22, C32, C33, C36, C40, C41: MPN (none) -> KGM15BR51A475KT
- C174: MPN (none) -> KGM15CR50J476MT
- D8, D9: MPN (none) -> ASCKC500NW5X4040
- FB4: MPN (none) -> 742792641
- J13: MPN (none) -> 87832-1420
- R2, R5, R51, R53, R54, R76, R81: MPN (none) -> SDR03EZPD4701
- R47: MPN (none) -> SDR03EZPD3300
- R77, R78, R79, R80: MPN (none) -> SDR03EZPD1000
- U15: MPN (none) -> IS25LP256DRMLETR
- U2: MPN (none) -> XC7A35T-1FTG256C
