File: hardware/MRC/mrc-fpga-config.kicad_sch (KiCad schematic)
At the start: 58 parts, among them J13 Conn_02x07_Odd_Even, U15 IS25LP256D-RMLE-TR, U2 XC7A35T-FTG256

Commit message: KiCAD schematic modification
Parts:
- C150, C175, C176, C177, C18, C181, C182, C183, C184, C185, C19, C20, C26, C30, C31, C35, C38, C87, C88: MPN 06035C474KAT4A -> C1623
- C172, C173, C178, C179, C186, C187, C21, C22, C32, C33, C36, C40, C41: MPN KGM15BR51A475KT -> C19666
- C174: MPN KGM15CR50J476MT -> C318632; Stock (none) -> Extended
- C180, C188, C25, C34, C42: MPN (none) -> C6663208; Stock (none) -> Extended
- D8, D9: MPN ASCKC500NW5X4040 -> C2286
- FB4: MPN 742792641 -> C14709
- J13: MPN 87832-1420 -> (none)
- R2, R5, R51, R53, R54, R76, R81: MPN SDR03EZPD4701 -> C23162
- R47: MPN SDR03EZPD3300 -> C23138
- R77, R78, R79, R80: MPN SDR03EZPD1000 -> C22775
- U15: MPN IS25LP256DRMLETR -> C2063380; Stock (none) -> Extended
- U2: MPN XC7A35T-1FTG256C -> C9900024150; Stock (none) -> Extended
