File: hardware/MRC/mrc-gradient.kicad_sch (KiCad schematic)
At the start: 15 parts, among them J22 SJ-63063B, J5 SJ-63063B, J7 SJ-63063B, U10 DRV8220, U22 DRV8220, U23 DRV8220, U24 DRV8220, U27 DRV8220, U28 DRV8220

Commit message: KiCAD schematic modification
Parts:
- C138, C196, C202: MPN 875585344003 -> C20040380; Stock (none) -> Extended
- J22, J5, J7: MPN SJ-63063B -> C4992577; Stock (none) -> Extended
- R25, R26, R30: MPN PWR221T-30-5R00J -> (none)
- U10, U22, U23, U24, U27, U28: MPN DRV8220DSGRCT -> C3681269; Stock (none) -> Extended
