File: hardware/MRC/mrc-magnet-interface.kicad_sch (KiCad schematic)
At the start: 3 parts, among them J9 RJ45_LED_Shielded

Commit message: Clean bill of materials
Parts:
- J9: MPN (none) -> RJHSE-5381
- R93, R94: MPN (none) -> SDR03EZPD4701
Changed lines of the file:
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@@
+			)
+		)
+		(property "MPN" "RJHSE-5381 "
+			(at 113.03 93.98 0)
+			(effects
+				(font
+					(size 1.27 1.27)
+				)
+				(hide yes)
 			)
 		)
@@
 			)
 		)
+		(property "MPN" "SDR03EZPD4701 "
+			(at 97.79 83.82 0)
+			(effects
+				(font
+					(size 1.27 1.27)
+				)
+				(hide yes)
+			)
+		)
 		(pin "1"
 		)
@@
 			)
 		)
+		(property "MPN" "SDR03EZPD4701 "
+			(at 97.79 99.06 0)
+			(effects
+				(font
+					(size 1.27 1.27)
+				)
+				(hide yes)
+			)
+		)
