File: hardware/MRC/mrc-magnet-interface.kicad_sch (KiCad schematic)
At the start: 3 parts, among them J9 RJ45_LED_Shielded

Commit message: KiCAD schematic modification
Parts:
- J9: MPN RJHSE-5381 -> C464586/C464587/C464588; Stock (none) -> Extended
- R93, R94: MPN SDR03EZPD4701 -> C23162
