File: hardware/MRC/mrc_fpga.kicad_sch (KiCad schematic)
At the start: 3 parts, among them J6 Conn_02x05_Odd_Even, U2 XC7A35T-FTG256

Commit message: Clean bill of materials
Parts:
- R27: MPN (none) -> CRCW06031K00DHEBP
- U2: MPN (none) -> XC7A35T-1FTG256C
Changed lines of the file:
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@@
+			)
+		)
+		(property "MPN" "XC7A35T-1FTG256C "
+			(at 77.47 97.79 90)
+			(effects
+				(font
+					(size 1.27 1.27)
+				)
+				(hide yes)
 			)
 		)
@@
 			)
 		)
+		(property "MPN" "XC7A35T-1FTG256C "
+			(at 209.55 91.44 0)
+			(effects
+				(font
+					(size 1.27 1.27)
+				)
+				(hide yes)
+			)
+		)
 		(pin "A10"
 		)
@@
 			)
 		)
+		(property "MPN" "CRCW06031K00DHEBP "
+			(at 142.24 54.61 0)
+			(effects
+				(font
+					(size 1.27 1.27)
+				)
+				(hide yes)
+			)
+		)
