File: hardware/MRC/mrc_fpga.kicad_sch (KiCad schematic)
At the start: 3 parts, among them J6 Conn_02x05_Odd_Even, U2 XC7A35T-FTG256

Commit message: KiCAD schematic modification
Parts:
- R27: MPN CRCW06031K00DHEBP -> C21190
- U2: MPN XC7A35T-1FTG256C -> C9900024150; Stock (none) -> Extended
Connections:
- net FPGASPI.SDO: now also J6.8 (Pin_8)
- net GND: no longer J6.8 (Pin_8)
- net IO0 renamed dbg_Reset
- net IO6 renamed dbg_Trigger
Other:
- moved on the sheet: J6
