File: hardware/MRC/mrc_usb.kicad_sch (KiCad schematic)
At the start: 45 parts, among them J14 GSB443133HR, U6 FT601Q, Y2 30Meg

Commit message: Clean bill of materials
Parts:
- C103, C104, C105, C109, C111, C113, C115, C118, C120, C122, C124, C126, C128, C130: MPN (none) -> C0603C104K1RACAUTO
- C106, C107: MPN (none) -> KGM15ACG1H180JT
- C110, C112, C114, C116, C125, C127, C129, C131: MPN (none) -> 06035C474KAT4A
- C117, C119, C121: MPN (none) -> KGM15AR71H682KT
- C123: MPN (none) -> KGM15BR51E105KM
- C132: MPN (none) -> KGM15BR51A475KT
- D2, D3: MPN (none) -> SJD12C05L01
- D4: MPN (none) -> SMLD12EN1WT86
- FB10: MPN (none) -> 742792641
- J14: MPN (none) -> GSB443133HR
- R52: MPN (none) -> ESR03EZPD4700
- R56: MPN (none) -> SDR03EZPD4701
- R57: MPN (none) -> CMP0603AFX-1002L
- R58, R59: MPN (none) -> SDR03EZPD1000
- R60: MPN (none) -> ERA-3ARB332V
- R64: MPN (none) -> ESR03EZPD1601
- U6: MPN (none) -> FT601Q-B-T
- Y2: MPN 830059646 -> 830059646
