File: hardware/MRC/mrc_usb.kicad_sch (KiCad schematic)
At the start: 45 parts, among them J14 GSB443133HR, U6 FT601Q, Y2 30Meg

Commit message: KiCAD schematic modification
Parts:
- added R61, R62, R63: 4.7k, Resistor_SMD:R_0603_1608Metric, symbol Device:R_Small
- C103, C104, C105, C109, C111, C113, C115, C118, C120, C122, C124, C126, C128, C130: MPN C0603C104K1RACAUTO -> C14663
- C106, C107: MPN KGM15ACG1H180JT -> C1647
- C110, C112, C114, C116, C125, C127, C129, C131: MPN 06035C474KAT4A -> C1623
- C117, C119, C121: MPN KGM15AR71H682KT -> C1631
- C123: MPN KGM15BR51E105KM -> C15849
- C132: MPN KGM15BR51A475KT -> C19666
- D2, D3: MPN SJD12C05L01 -> (none)
- D4: MPN SMLD12EN1WT86 -> C2290
- FB10: MPN 742792641 -> C14709
- J14: MPN GSB443133HR -> C5428289(need to confirm); Stock (none) -> Extended
- R52: MPN ESR03EZPD4700 -> C23179
- R56: MPN SDR03EZPD4701 -> C23162
- R57: MPN CMP0603AFX-1002L -> C25804
- R58, R59: MPN SDR03EZPD1000 -> C22775
- R60: MPN ERA-3ARB332V -> C22978
- R64: MPN ESR03EZPD1601 -> C22847; Stock (none) -> Extended
- U6: MPN FT601Q-B-T -> C1550513; Stock (none) -> Extended
- Y2: MPN 830059646 -> C20885054; Stock (none) -> Extended
Connections:
- net +3V3: now also R61.1, R62.1, R63.1
- net USB_~{RESET}: now also R62.2
- net USB_~{SIWU}: now also R61.2
- net USB_~{WAKEUP}: now also R63.2
