File: hardware/MRC/MR-Core.kicad_sch (KiCad schematic)
At the start: 8 parts, among them J1 Conn_Coaxial, J16 Conn_Coaxial, J17 Conn_Coaxial, J18 Conn_Coaxial, J2 Conn_Coaxial, J3 Conn_Coaxial, J4 Conn_Coaxial, J8 Conn_Coaxial

Commit message: KiCAD schematic modification
Parts:
- J1, J2, J3, J4: MPN 73415-1471 -> C588477; Stock (none) -> Extended
- J16, J17, J18, J8: MPN CONSMA013.062-G -> C588477; Stock (none) -> Extended
