File: hardware/MRC/mrc_controller.kicad_sch (KiCad schematic)
At the start: 72 parts, among them J10 Conn_02x04_Odd_Even, J11 Conn_02x07_Odd_Even, J15 RJ45_Wuerth_7499010121A, J23 USB_B_Mini, J24 Micro_SD_Card_Det_Hirose_DM3AT, U13 LAN8742A, U17 USBLC6-4SC6, U9 STM32F767ZITx, X1 50M, Y1 X53T-C20SSA-25.000MHz, Y3 32.768k

Commit message: KiCAD schematic modification
Parts:
- C100, C101: MPN KGM15BR50J225KT -> C23630
- C102, C140, C141, C142, C143, C144, C145, C146, C151, C152, C156, C163, C165, C167, C205, C209, C97, C99: MPN C0603C104K1RACAUTO -> C14663
- C147, C153, C164, C166, C208, C96, C98: MPN KGM15BR51E105KM -> C15849
- C148, C149: MPN KGM15ACG2A100FT -> C1634
- C203, C204: MPN C0603C300J5G -> C1658
- C206: MPN KGM21AR50J106KU -> C96446
- C207: MPN KGM15AR71H471KT -> C1620
- FB1, FB11, FB3: MPN 742792641 -> C14709
- J11: MPN FTSH10701FDVKP -> (none)
- J15: MPN 7499010121A -> C5451791; Stock (none) -> Extended
- J23: MPN 65100516121 -> C5120592; Stock (none) -> Extended
- J24: MPN DM3BT-DSF-PEJS -> C597972; Stock (none) -> Extended
- R13, R24, R3, R32, R33, R35, R38, R39, R4, R46, R48: MPN CMP0603AFX-1002L -> C25804
- R29, R34, R36, R37: MPN SDR03EZPF33R0 -> C23140
- R40, R41, R42, R43: MPN SDR03EZPF51R0 -> C23197
- R44: MPN SDR03EZPF47R0 -> C23182
- R45, R87: MPN ERJ-3GEYJ271V -> C22966
- R89: MPN KTR03EZPF1212 -> C22864; Stock (none) -> Extended
- U13: MPN LAN8742AI-CZ-TR -> C621425; Stock (none) -> Extended
- U17: MPN USBLC6-4SC6 -> C5197386; Stock (none) -> Extended
- U9: MPN STM32F767ZIT6 -> C90235; Stock (none) -> Extended
- X1: MPN 2520MV-500-DN-TR -> C17348430; Stock (none) -> Extended
- Y1: MPN (none) -> C717795; Stock (none) -> Extended
- Y3: MPN 202257-MC01 -> C5341287/C5341288; Stock (none) -> Extended
Connections:
- net uC_IO0 renamed dbg_Reset
- net uC_IO4 renamed dbg_Trigger
